File: kicad/main/az030.kicad_pcb (KiCad board)
At the start: 4 copper layers, 211.4 x 139.8 mm, 37 parts, among them J1 ATX-24, J10 Bus_PCI_32bit_Universal, J2 Conn_01x02_Pin, J3 LED, J4 Conn_01x03_Pin, J5 Conn_01x03_Pin, J6 Conn_01x03_Pin, J7 Conn_01x03_Pin, J8 DE9_Pins_MountingHoles, J9 DB25_Pins_MountingHoles, SW1 SW_Push, U1 MC68030RC_PGA, U2 74HC74, U3 W65C22SxP, U4 W65C22SxP, U5 GAL16V8, U6 GAL16V8, U7 CY62256-70PC, Y1 CXO_DIP8

Commit message: ygffd
Parts:
- removed F3, F4: 3a, Fuse:Fuse_Blade_ATO_directSolder
- removed J10: Bus_PCI_32bit_Universal, Connector_PCBEdge:Samtec_MECF-60-01-L-DV-WT_2x60_P1.27mm_Polarized_Socket_Horizontal
- removed J6, J7: Conn_01x03_Pin, Connector:FanPinHeader_1x03_P2.54mm_Vertical
- removed J8: DE9_Pins_MountingHoles, Connector_Dsub:DSUB-9_Pins_Horizontal_P2.77x2.84mm_EdgePinOffset4.94mm_Housed_MountingHolesOffset4.94mm
- removed J9: DB25_Pins_MountingHoles, Connector_Dsub:DSUB-25_Pins_Horizontal_P2.77x2.84mm_EdgePinOffset4.94mm_Housed_MountingHolesOffset4.94mm
- removed REF** (x4): MountingHole_2.2mm_M2_Pad, MountingHole:MountingHole_2.2mm_M2_Pad
- removed U3, U4: W65C22SxP, Package_DIP:DIP-40_W15.24mm
- removed U8: ~, Package_DIP:DIP-48_W15.24mm_LongPads
- removed U9: ~, Connector_PCBEdge:Samtec_MECF-40-01-L-DV-WT_2x40_P1.27mm_Polarized_Socket_Horizontal
- added H1: MountingHole_Pad, MountingHole:MountingHole_4mm_Pad, F.Cu at (95.0, 65.0)
- added H2: MountingHole_Pad, MountingHole:MountingHole_4mm_Pad, F.Cu at (95.0, 195.0)
- added H3: MountingHole_Pad, MountingHole:MountingHole_4mm_Pad, F.Cu at (295.0, 65.0)
- added H4: MountingHole_Pad, MountingHole:MountingHole_4mm_Pad, F.Cu at (290.0, 185.0)
- added H5: MountingHole_Pad, MountingHole:MountingHole_4mm_Pad, F.Cu at (144.3, 144.3)
- added J11: VERA, Connector_PinSocket_2.54mm:PinSocket_2x12_P2.54mm_Vertical, F.Cu at (127.5, 89.7)
- added R10: 10k, Resistor_SMD:R_0603_1608Metric, F.Cu at (224.2, 107.5)
- added R9: 10k, Resistor_SMD:R_0603_1608Metric, F.Cu at (224.2, 105.0)
- J4: value Conn_01x03_Pin -> DE9_Socket_MountingHoles; footprint Connector:FanPinHeader_1x03_P2.54mm_Vertical -> Connector_Dsub:DSUB-9_Socket_Horizontal_P2.77x2.84mm_EdgePinOffset4.94mm_Housed_MountingHolesOffset4.94mm
- J5: value Conn_01x03_Pin -> DB25_Socket_MountingHoles; footprint Connector:FanPinHeader_1x03_P2.54mm_Vertical -> Connector_Dsub:DSUB-25_Socket_Horizontal_P2.77x2.84mm_EdgePinOffset4.94mm_Housed_MountingHolesOffset4.94mm
- R1: moved to F.Cu
- R8: moved to B.Cu
- U2: footprint Package_DIP:DIP-14_W7.62mm_LongPads -> Package_DIP:DIP-14_W7.62mm
- moved J3 132.1 mm to (295.0, 165.0), turned to 0 degrees
- moved R7 125.4 mm to (290.0, 165.0), turned to 180 degrees
- moved U7 119.1 mm to (239.8, 92.4)
- moved J2 117.1 mm to (295.0, 152.5), turned to 0 degrees
- moved J4 75.5 mm to (97.8, 150.5), turned to -90 degrees
- moved J1 68.3 mm to (287.7, 100.0), turned to -90 degrees
- moved JP1 67.2 mm to (184.8, 130.2), turned to 180 degrees
- moved R8 62.4 mm to (163.8, 125.2), turned to 90 degrees
- moved U2 56.2 mm to (167.1, 114.9)
- moved F2 56.1 mm to (269.3, 145.0), turned to 180 degrees
- moved U5 45.5 mm to (197.4, 135.0)
- moved U6 44.7 mm to (211.2, 135.0)
- moved R4 38.4 mm to (206.8, 106.2)
- moved R5 38.2 mm to (217.8, 109.6), turned to -90 degrees
- moved R2 37.7 mm to (192.8, 108.2)
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Connections:
- J1 pad 1: Net-(F3-Pad1) -> unconnected-(J1-+3.3V-Pad1)
- J1 pad 10: Net-(F4-Pad1) -> unconnected-(J1-+12V-Pad10)
- J1 pad 11: Net-(F4-Pad1) -> unconnected-(J1-+12V-Pad10)_1
- J1 pad 12: Net-(F3-Pad1) -> unconnected-(J1-+3.3V-Pad1)_3
- J1 pad 13: Net-(F3-Pad1) -> unconnected-(J1-+3.3V-Pad1)_1
- J1 pad 2: Net-(F3-Pad1) -> unconnected-(J1-+3.3V-Pad1)_2
- J4 pad 1: GND -> unconnected-(J4-Pad1)
- J4 pad 2: +12V -> unconnected-(J4-Pad2)
- J5 pad 1: GND -> unconnected-(J5-Pad1)
- J5 pad 2: +12V -> unconnected-(J5-Pad2)
- U1 pad E2: GND -> /CPU/VERA/IRQ
- U1 pad F1: DSACK0 -> Net-(U1-DSACK0)
- U1 pad G12: IPL2 -> unconnected-(U1-IPL2-PadG12)
- U1 pad G13: IPL1 -> unconnected-(U1-IPL1-PadG13)
- U1 pad G2: DSACK1 -> Net-(U1-DSACK1)
- U1 pad M2: ECS -> unconnected-(U1-ECS-PadM2)
- U2 pad 3: ECS -> unconnected-(U2A-C-Pad3)
Routing:
- net RAM0: track 126.3 -> 0.00 mm, vias 3 -> 0
- net /CPU/A0: track 106.8 -> 0.00 mm
- net R~{W}: track 105.3 -> 0.00 mm, vias 1 -> 0
- net /CPU/A4: track 97.1 -> 0.00 mm, vias 3 -> 0
- net Net-(F3-Pad1): track 96.9 -> 0.00 mm, vias 2 -> 0
- net /CPU/D0: track 91.6 -> 0.00 mm, vias 1 -> 0
- net /CPU/A6: track 76.4 -> 0.00 mm, vias 1 -> 0
- net /CPU/D1: track 75.2 -> 0.00 mm
- net SIZ1: track 74.0 -> 0.00 mm
- net /CPU/D7: track 72.1 -> 0.00 mm
- net DSACK1: track 68.0 -> 0.00 mm, vias 1 -> 0
- net DSACK0: track 65.7 -> 0.00 mm, vias 2 -> 0
- net /CPU/D2: track 65.5 -> 0.00 mm, vias 3 -> 0
- net STERM: track 64.2 -> 0.00 mm, vias 1 -> 0
- net /CPU/A3: track 62.4 -> 0.00 mm, vias 1 -> 0
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- added copper zone on In1.Cu, net (none)
- added copper zone on In2.Cu, net (none)
- removed copper zone on In2.Cu, net +12V
- removed copper zone on In1.Cu, net +3.3V
Other:
- board size 211.4 x 139.8 mm -> 210 x 139.8 mm
- board text removed: "+ -"
- board text removed: "16-50MHz"
- board text removed: "Fan Headers might only use one icl"
- board text removed: "GLUE Logic"
- board text removed: "Power LED"
- board text removed: "Power Switch"
- board text removed: "all of these resistors here are 10k"
