File: kicad/main/az030.kicad_pcb (KiCad board)
At the start: 2 copper layers, 7 parts, among them U1 MC68030RC_PGA, U3 W65C22SxP, U4 W65C22SxP, Y1 CXO_DIP8

Commit message: so much shit done holy
Parts:
- added C1: 100n, Capacitor_SMD:C_0201_0603Metric, B.Cu at (232.3, 98.5)
- added C2: 10u, Capacitor_SMD:C_0201_0603Metric, B.Cu at (228.0, 92.0)
- added C3: 100n, Capacitor_SMD:C_0201_0603Metric, B.Cu at (227.0, 102.5)
- added F2: 5a, Fuse:Fuse_Blade_ATO_directSolder, F.Cu at (273.1, 89.0)
- added F3: 3a, Fuse:Fuse_Blade_ATO_directSolder, F.Cu at (265.6, 89.0)
- added F4: 3a, Fuse:Fuse_Blade_ATO_directSolder, B.Cu at (258.0, 89.0)
- added J1: ATX-24, Connector_Molex:Molex_Mini-Fit_Jr_5569-24A2_2x12_P4.20mm_Horizontal, F.Cu at (225.8, 71.1)
- added J2: Conn_01x02_Pin, Connector_PinHeader_2.54mm:PinHeader_1x02_P2.54mm_Vertical, F.Cu at (216.0, 66.0)
- added J3: LED, Connector_PinHeader_2.54mm:PinHeader_1x02_P2.54mm_Vertical, F.Cu at (207.5, 66.0)
- added J4: Conn_01x03_Pin, Connector:FanPinHeader_1x03_P2.54mm_Vertical, F.Cu at (95.8, 132.5)
- added J5: Conn_01x03_Pin, Connector:FanPinHeader_1x03_P2.54mm_Vertical, F.Cu at (95.8, 145.0)
- added J6: Conn_01x03_Pin, Connector:FanPinHeader_1x03_P2.54mm_Vertical, F.Cu at (95.8, 157.5)
- added J7: Conn_01x03_Pin, Connector:FanPinHeader_1x03_P2.54mm_Vertical, F.Cu at (95.8, 170.0)
- added J8: Conn_01x04_Pin, Connector_PinHeader_2.54mm:PinHeader_1x04_P2.54mm_Vertical, F.Cu at (220.0, 92.0)
- added R1: 10k, Resistor_SMD:R_1206_3216Metric, B.Cu at (167.9, 84.0)
- added R2: 10k, Resistor_SMD:R_1206_3216Metric, B.Cu at (162.9, 85.0)
- added R3: 10k, Resistor_SMD:R_1206_3216Metric, B.Cu at (188.9, 78.0)
- added R4: 10k, Resistor_SMD:R_1206_3216Metric, B.Cu at (176.9, 82.0)
- added R5: 10k, Resistor_SMD:R_1206_3216Metric, B.Cu at (188.5, 85.0)
- added R6: 10k, Resistor_SMD:R_1206_3216Metric, B.Cu at (185.4, 106.5)
- added R7: 330, Resistor_THT:R_Axial_DIN0204_L3.6mm_D1.6mm_P7.62mm_Horizontal, F.Cu at (208.0, 70.2)
- added REF**: MountingHole_2.2mm_M2_Pad, MountingHole:MountingHole_2.2mm_M2_Pad, F.Cu at (92.0, 63.5)
- added REF**: MountingHole_2.2mm_M2_Pad, MountingHole:MountingHole_2.2mm_M2_Pad, F.Cu at (92.0, 285.5)
- added REF**: MountingHole_2.2mm_M2_Pad, MountingHole:MountingHole_2.2mm_M2_Pad, F.Cu at (390.0, 63.5)
- added REF**: MountingHole_2.2mm_M2_Pad, MountingHole:MountingHole_2.2mm_M2_Pad, F.Cu at (390.0, 285.5)
- added SW1: SW_Push, Button_Switch_THT:SW_PUSH_6mm, F.Cu at (189.7, 89.3)
- added U5: XC9572XL-10VQG64C, Package_QFP:TQFP-64_10x10mm_P0.5mm, F.Cu at (228.8, 95.7)
- moved F1 177.9 mm to (368.0, 88.7), turned to 180 degrees
- moved D1 177.7 mm to (368.1, 81.5), turned to 180 degrees
- moved U2 165.2 mm to (382.5, 79.8)
- moved U4 56.0 mm to (96.2, 68.6)
- moved U1 56.0 mm to (169.8, 87.5)
- moved U3 56.0 mm to (124.1, 68.6)
- moved Y1 56.0 mm to (200.3, 100.2)
Connections:
- net Net-(U1-CLKIN) renamed /CPU/CLOCK
- U1 pad A1: unconnected-(U1-BR-PadA1) -> Net-(U1-BR)
- U1 pad F12: unconnected-(U1-RESET-PadF12) -> Net-(U1-HLT)
- U1 pad H1: unconnected-(U1-BERR-PadH1) -> Net-(U1-BERR)
- U1 pad H12: unconnected-(U1-CDIS-PadH12) -> Net-(U1-CDIS)
- U1 pad H2: unconnected-(U1-HLT-PadH2) -> Net-(U1-HLT)
- U1 pad K1: unconnected-(U1-CBREQ-PadK1) -> Net-(U1-CBREQ)
- U1 pad L1: unconnected-(U1-CIIN-PadL1) -> Net-(U1-CIIN)
- U1 pad L3: unconnected-(U1-R_W-PadL3) -> /CPU/R~{W}
- U3 pad 22: unconnected-(U3-R/~{W}-Pad22) -> /Peripheral Management/R~{W}
- U4 pad 22: unconnected-(U4-R/~{W}-Pad22) -> /Peripheral Management/R~{W}
Routing:
- net Net-(F2-Pad1): track 0.00 -> 123.9 mm, vias 0 -> 1
- net Net-(F3-Pad1): track 0.00 -> 96.9 mm, vias 0 -> 2
- net Net-(J1-PWR_OK): track 0.00 -> 53.5 mm, vias 0 -> 1
- net Net-(U1-HLT): track 0.00 -> 51.4 mm
- net Net-(F4-Pad1): track 0.00 -> 47.5 mm
- net Net-(J1-PS_ON#): track 0.00 -> 29.3 mm
- net /CPU/CLOCK: track 0.00 -> 24.1 mm
- net /CPU/RESET: track 0.00 -> 23.3 mm
- net Net-(J8-Pin_4): track 0.00 -> 18.6 mm
- net Net-(J8-Pin_3): track 0.00 -> 9.51 mm
- net Net-(J8-Pin_2): track 0.00 -> 9.33 mm, vias 0 -> 1
- net Net-(U1-CBREQ): track 0.00 -> 7.61 mm
- net Net-(J8-Pin_1): track 0.00 -> 7.28 mm
- net Net-(U1-CDIS): track 0.00 -> 5.19 mm
- net Net-(J3-Pin_1): track 0.00 -> 4.38 mm
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- added copper zone on In2.Cu, net +12V
- added copper zone on In1.Cu, net +3.3V
- added copper zone on B.Cu, net +5V
- added copper zone on F.Cu, net GND
Other:
- board outline added: 304.8 x 228.6 mm
- copper layers 2 -> 4
- board text added: "+ -"
- board text added: "16-50MHz"
- board text added: "Fan Headers might only use one icl"
- board text added: "GLUE Logic"
- board text added: "JTAG"
- board text added: "Power LED"
- board text added: "Power Switch"
- board text added: "all of these resistors here are 10k"

Commit message: fjfjkdsldkjjfds
Parts:
- removed C1, C3: 100n, Capacitor_SMD:C_0201_0603Metric
- removed C2: 10u, Capacitor_SMD:C_0201_0603Metric
- removed D1: 1n4001, Diode_THT:D_DO-41_SOD81_P10.16mm_Horizontal
- removed F1: 1a, Fuse:Fuse_Littelfuse-LVR100
- added J10: Bus_PCI_32bit_Universal, Connector_PCBEdge:Samtec_MECF-60-01-L-DV-WT_2x60_P1.27mm_Polarized_Socket_Horizontal, F.Cu at (246.9, 153.1)
- added J9: DB25_Pins_MountingHoles, Connector_Dsub:DSUB-25_Pins_Horizontal_P2.77x2.84mm_EdgePinOffset4.94mm_Housed_MountingHolesOffset4.94mm, F.Cu at (151.2, 192.2)
- added JP1: RUN, TestPoint:TestPoint_2Pads_Pitch5.08mm_Drill1.3mm, F.Cu at (182.5, 63.0)
- added R8: 10k, Resistor_SMD:R_1206_3216Metric, F.Cu at (187.5, 67.5)
- added U6: GAL16V8, Package_DIP:DIP-20_W7.62mm_LongPads, F.Cu at (225.0, 92.5)
- added U7: CY62256-70PC, Package_DIP:DIP-28_W15.24mm, F.Cu at (123.4, 67.1)
- added U8: ~, Package_DIP:DIP-48_W15.24mm_LongPads, F.Cu at (170.0, 115.8)
- added U9: ~, Connector_PCBEdge:Samtec_MECF-40-01-L-DV-WT_2x40_P1.27mm_Polarized_Socket_Horizontal, F.Cu at (226.9, 165.7)
- J8: value Conn_01x04_Pin -> DE9_Pins_MountingHoles; footprint Connector_PinHeader_2.54mm:PinHeader_1x04_P2.54mm_Vertical -> Connector_Dsub:DSUB-9_Pins_Horizontal_P2.77x2.84mm_EdgePinOffset4.94mm_Housed_MountingHolesOffset4.94mm
- U2: value ~ -> 74HC74; footprint Connector_IDC:IDC-Header_2x25_P2.54mm_Horizontal -> Package_DIP:DIP-14_W7.62mm_LongPads
- U5: value XC9572XL-10VQG64C -> GAL16V8; footprint Package_QFP:TQFP-64_10x10mm_P0.5mm -> Package_DIP:DIP-20_W7.62mm_LongPads
- moved U2 190.6 mm to (192.5, 64.8)
- moved J8 147.4 mm to (112.0, 192.2)
- moved REF** 129.1 mm to (296.5, 196.5)
- moved REF** 93.5 mm to (296.5, 63.5)
- moved REF** 89.0 mm to (92.0, 196.5)
- moved J4 57.5 mm to (95.0, 75.1)
- moved J5 57.5 mm to (95.0, 87.5)
- moved J6 57.5 mm to (95.0, 100.0)
- moved J7 57.5 mm to (95.0, 112.5)
- moved U4 56.5 mm to (124.8, 117.3)
- moved U3 54.1 mm to (147.5, 117.4)
- moved U5 15.7 mm to (213.4, 92.5), turned to 0 degrees
Connections:
- net /CPU/CLOCK renamed CLOCK
- J8 pad 1: Net-(J8-Pin_1) -> unconnected-(J8-Pad1)
- J8 pad 2: Net-(J8-Pin_2) -> unconnected-(J8-Pad2)
- J8 pad 3: Net-(J8-Pin_3) -> unconnected-(J8-Pad3)
- J8 pad 4: Net-(J8-Pin_4) -> unconnected-(J8-Pad4)
- R1 pad 2: /CPU/RESET -> RESET
- SW1 pad 1: /CPU/RESET -> RESET
- SW1 pad 2: Net-(U1-HLT) -> Net-(U1-RESET)
- U1 pad C1: unconnected-(U1-FC1-PadC1) -> FC1
- U1 pad D1: unconnected-(U1-FC2-PadD1) -> FC2
- U1 pad D2: unconnected-(U1-FC0-PadD2) -> FC0
- U1 pad E2: unconnected-(U1-AVEC-PadE2) -> GND
- U1 pad F1: unconnected-(U1-DSACK0-PadF1) -> DSACK0
- U1 pad F12: Net-(U1-HLT) -> Net-(U1-RESET)
- U1 pad G1: unconnected-(U1-STERM-PadG1) -> STERM
- U1 pad G12: unconnected-(U1-IPL2-PadG12) -> IPL2
- U1 pad G13: unconnected-(U1-IPL1-PadG13) -> IPL1
- U1 pad G2: unconnected-(U1-DSACK1-PadG2) -> DSACK1
- U1 pad H13: unconnected-(U1-IPL0-PadH13) -> +5V
- U1 pad H2: Net-(U1-HLT) -> Net-(JP1-A)
- U1 pad J2: unconnected-(U1-AS-PadJ2) -> AS
- U1 pad K2: unconnected-(U1-DS-PadK2) -> DS
- U1 pad K3: unconnected-(U1-SIZ1-PadK3) -> SIZ1
- U1 pad L2: unconnected-(U1-SIZ0-PadL2) -> SIZ0
- U1 pad L3: /CPU/R~{W} -> R~{W}
- U1 pad M2: unconnected-(U1-ECS-PadM2) -> ECS
- U2 pad 1: (no net) -> RESET
- U2 pad 10: unconnected-(U2-DB4-Pad10) -> (no net)
- U2 pad 12: unconnected-(U2-DB5-Pad12) -> (no net)
- U2 pad 14: unconnected-(U2-DB6-Pad14) -> +5V
- U2 pad 2: unconnected-(U2-DB0-Pad2) -> Net-(U2A-D)
- U2 pad 3: (no net) -> ECS
- U2 pad 4: unconnected-(U2-DB1-Pad4) -> Net-(U2A-~{S})
- U2 pad 5: (no net) -> Net-(JP1-B)
- U2 pad 6: unconnected-(U2-DB2-Pad6) -> Net-(U2A-D)
- U2 pad 7: (no net) -> GND
- U2 pad 8: unconnected-(U2-DB3-Pad8) -> (no net)
- U5 pad 1: unconnected-(U5-I/O-Pad1) -> /CPU/A1
- U5 pad 10: unconnected-(U5-I/O-Pad10) -> GND
- U5 pad 13: unconnected-(U5-I/O-Pad13) -> RAM0
- U5 pad 14: Net-(C3-Pad1) -> RAM1
- U5 pad 15: unconnected-(U5-I/O/GCK1-Pad15) -> RAM2
- U5 pad 16: unconnected-(U5-I/O/GCK2-Pad16) -> RAM3
- U5 pad 17: unconnected-(U5-I/O/GCK3-Pad17) -> ROM
- U5 pad 18: unconnected-(U5-I/O-Pad18) -> UART
- U5 pad 19: unconnected-(U5-I/O-Pad19) -> EXT
- U5 pad 2: unconnected-(U5-I/O/GTS2-Pad2) -> /CPU/A0
- U5 pad 20: unconnected-(U5-I/O-Pad20) -> +5V
- U5 pad 3: Net-(C1-Pad1) -> /CPU/A19
- U5 pad 4: unconnected-(U5-I/O-Pad4) -> /CPU/A20
- U5 pad 5: unconnected-(U5-I/O/GTS1-Pad5) -> /CPU/A25
- U5 pad 6: unconnected-(U5-I/O-Pad6) -> SIZ0
- U5 pad 7: unconnected-(U5-I/O-Pad7) -> SIZ1
- U5 pad 8: unconnected-(U5-I/O-Pad8) -> AS
Routing:
- net RAM0: track 0.00 -> 126.3 mm, vias 0 -> 3
- net /CPU/A0: track 0.00 -> 106.8 mm
- net R~{W}: track 0.00 -> 105.3 mm, vias 0 -> 1
- net /CPU/A4: track 0.00 -> 97.1 mm, vias 0 -> 3
- net /CPU/D0: track 0.00 -> 91.6 mm, vias 0 -> 1
- net /CPU/A6: track 0.00 -> 76.4 mm, vias 0 -> 1
- net /CPU/D1: track 0.00 -> 75.2 mm
- net SIZ1: track 0.00 -> 74.0 mm
- net /CPU/D7: track 0.00 -> 72.1 mm
- net DSACK1: track 0.00 -> 68.0 mm, vias 0 -> 1
- net DSACK0: track 0.00 -> 65.7 mm, vias 0 -> 2
- net /CPU/D2: track 0.00 -> 65.5 mm, vias 0 -> 3
- net STERM: track 0.00 -> 64.2 mm, vias 0 -> 1
- net /CPU/A3: track 0.00 -> 62.4 mm, vias 0 -> 1
- net /CPU/A12: track 0.00 -> 60.3 mm, vias 0 -> 1
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Other:
- board size 304.8 x 228.6 mm -> 211.4 x 139.8 mm
- board text removed: "JTAG"

Commit message: remove some stuff
Parts:
- removed J10: Bus_PCI_32bit_Universal, Connector_PCBEdge:Samtec_MECF-60-01-L-DV-WT_2x60_P1.27mm_Polarized_Socket_Horizontal
- removed U9: ~, Connector_PCBEdge:Samtec_MECF-40-01-L-DV-WT_2x40_P1.27mm_Polarized_Socket_Horizontal
- added C1: 1u, Capacitor_SMD:C_0805_2012Metric, F.Cu at (214.0, 157.0)
- added C2: 1u, Capacitor_SMD:C_0805_2012Metric, F.Cu at (214.0, 164.0)
- added C3: 1u, Capacitor_SMD:C_0805_2012Metric, B.Cu at (220.0, 159.0)
- added C4: 1u, Capacitor_SMD:C_0805_2012Metric, B.Cu at (220.0, 169.1)
- added J11: PS/2, Footprints:Connector_Mini-DIN_Female_6Pin_2rows, F.Cu at (209.8, 191.3)
- added U10: 74AHC595, Package_DIP:DIP-16_W7.62mm_LongPads, F.Cu at (188.4, 154.9)
- added U11: 74AHC04, Package_DIP:DIP-14_W7.62mm_LongPads, F.Cu at (200.0, 154.9)
- added U12: MAX232, Package_DIP:DIP-16_W7.62mm_LongPads, F.Cu at (217.4, 155.0)
Routing:
- net Net-(U12-C1-): track 0.00 -> 4.26 mm
- net Net-(U12-C1+): track 0.00 -> 3.81 mm
- net Net-(U12-C2+): track 0.00 -> 3.56 mm
- net Net-(U12-C2-): track 0.00 -> 3.47 mm
- net Net-(U12-VS+): track 0.00 -> 2.83 mm
- net Net-(U12-VS-): track 0.00 -> 2.79 mm
