File: kicad/main/az030.kicad_sch (KiCad schematic)
At the start: 0 parts

Commit message: remove some stuff
Other:
- sheet Input And Output ports: added PS/2 D0, PS/2 D1, PS/2 D2, PS/2 D3, PS/2 D4, PS/2 D5, PS/2 D6, PS/2 D7; removed none
Changed lines of the file:
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@@
 	)
 	(sheet
-		(at 49.53 82.55)
+		(at 29.21 80.01)
 		(size 12.7 3.81)
 		(exclude_from_sim no)
@@
 		)
 		(property "Sheetname" "SIMMs"
-			(at 49.53 81.8384 0)
+			(at 29.21 79.2984 0)
 			(show_name no)
 			(do_not_autoplace no)
@@
 		)
 		(property "Sheetfile" "simms.kicad_sch"
-			(at 49.53 86.9446 0)
+			(at 29.21 84.4046 0)
 			(show_name no)
 			(do_not_autoplace no)
@@
 	)
 	(sheet
-		(at 102.87 78.74)
-		(size 12.7 3.81)
+		(at 96.52 67.31)
+		(size 21.59 22.86)
 		(exclude_from_sim no)
 		(in_bom yes)
@@
 		)
 		(property "Sheetname" "Input And Output"
-			(at 102.87 78.0284 0)
+			(at 96.52 66.5984 0)
 			(show_name no)
 			(do_not_autoplace no)
@@
 		)
 		(property "Sheetfile" "io.kicad_sch"
-			(at 102.87 83.1346 0)
+			(at 96.52 90.7546 0)
 			(show_name no)
 			(do_not_autoplace no)
@@
 				)
 				(justify left top)
+			)
+		)
+		(pin "PS{slash}2 D0" input
+			(at 96.52 68.58 180)
+			(effects
+				(font
+					(size 1.27 1.27)
+				)
+				(justify left)
+			)
+		)
+		(pin "PS{slash}2 D1" input
+			(at 96.52 71.12 180)
+			(effects
+				(font
+					(size 1.27 1.27)
+				)
+				(justify left)
+			)
+		)
+		(pin "PS{slash}2 D2" input
+			(at 96.52 73.66 180)
+			(effects
+				(font
+					(size 1.27 1.27)
+				)
+				(justify left)
+			)
+		)
+		(pin "PS{slash}2 D3" input
+			(at 96.52 76.2 180)
+			(effects
+				(font
+					(size 1.27 1.27)
+				)
+				(justify left)
+			)
+		)
+		(pin "PS{slash}2 D4" input
+			(at 96.52 78.74 180)
+			(effects
+				(font
+					(size 1.27 1.27)
+				)
+				(justify left)
+			)
+		)
+		(pin "PS{slash}2 D5" input
+			(at 96.52 81.28 180)
+			(effects
+				(font
+					(size 1.27 1.27)
+				)
+				(justify left)
+			)
+		)
+		(pin "PS{slash}2 D6" input
+			(at 96.52 83.82 180)
+			(effects
+				(font
+					(size 1.27 1.27)
+				)
+				(justify left)
+			)
+		)
+		(pin "PS{slash}2 D7" input
+			(at 96.52 86.36 180)
+			(effects
+				(font
+					(size 1.27 1.27)
+				)
+				(justify left)
 			)
 		)
@@
 	)
 	(sheet
-		(at 101.6 88.9)
-		(size 12.7 3.81)
+		(at 104.14 110.49)
+		(size 27.94 13.97)
 		(exclude_from_sim no)
 		(in_bom yes)
@@
 		)
 		(property "Sheetname" "Peripheral Management"
-			(at 101.6 88.1884 0)
+			(at 104.14 109.7784 0)
 			(show_name no)
 			(do_not_autoplace no)
@@
 		)
 		(property "Sheetfile" "perMan.kicad_sch"
-			(at 101.6 93.2946 0)
+			(at 104.14 125.0446 0)
 			(show_name no)
 			(do_not_autoplace no)
@@
 	)
 	(sheet
-		(at 54.61 93.98)
+		(at 29.21 71.12)
 		(size 12.7 3.81)
 		(exclude_from_sim no)
@@
 		)
 		(property "Sheetname" "Built-in Memory"
-			(at 54.61 93.2684 0)
+			(at 29.21 70.4084 0)
 			(show_name no)
 			(do_not_autoplace no)
@@
 		)
 		(property "Sheetfile" "biRAM.kicad_sch"
-			(at 54.61 98.3746 0)
-			(show_name no)
-			(do_not_autoplace no)
+			(at 29.21 75.5146 0)
+			(show_name no)
+			(do_not_autoplace no)
