File: kicad/main/cpu.kicad_sch (KiCad schematic)
At the start: 2 parts, among them U1 MC68030RC_PGA, Y1 CXO_DIP8

Commit message: guhdwhudsa
Connections:
- net R~{W}: now reaches U1.L3 (R_W)
Changed lines of the file:
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@@
+	(wire
+		(pts
+			(xy 101.6 111.76) (xy 107.95 111.76)
+		)
+		(stroke
+			(width 0)
+			(type default)
+		)
+	)
 	(wire
 		(pts
@@
 		)
 	)
+	(label "R~{W}"
+		(at 101.6 111.76 180)
+		(effects
+			(font
+				(size 1.27 1.27)
+			)
+			(justify right bottom)
+		)
+	)

Commit message: so much shit done holy
Parts:
- added R1, R2, R3, R4, R5, R6: 10k, Resistor_SMD:R_1206_3216Metric, symbol Device:R_US
- added SW1: SW_Push, Button_Switch_THT:SW_PUSH_6mm, symbol Switch:SW_Push
Connections:
- net +5V: now also R1.1, R2.2, R3.2, R4.2, R5.2, R6.1
- net CLOCK: now reaches U1.E1 (CLKIN), Y1.5 (OUT)
- net at U1.A1 (BR): now also R6.2
- net at U1.F12 (RESET): now also U1.H2 (HLT), SW1.2
- net at U1.H1 (BERR): now also R5.1
- net at U1.H12 (CDIS): now also R2.1
- net at U1.K1 (CBREQ): now also R4.1
- net at U1.L1 (CIIN): now also R3.1
- new net RESET: R1.2, SW1.1
- no-connect marks 5 -> 15
Other:
- title: (none) -> CPU

Commit message: fjfjkdsldkjjfds
Parts:
- added JP1: RUN, TestPoint:TestPoint_2Pads_Pitch5.08mm_Drill1.3mm, symbol Jumper:Jumper_2_Open
- added R8: 10k, Resistor_SMD:R_1206_3216Metric, symbol Device:R_US
- added U2: 74HC74, Package_DIP:DIP-14_W7.62mm_LongPads, symbol 74xx:74HC74
- added U7: CY62256-70PC, Package_DIP:DIP-28_W15.24mm, symbol Memory_RAM:CY62256-70PC
Connections:
- net +5V: now also U1.H13 (IPL0), R8.1, U2.14 (VCC), U7.28 (VCC)
- net A0: now also U7.10 (A0)
- net A1: now also U7.9 (A1)
- net A10: now also U7.21 (A10)
- net A11: now also U7.23 (A11)
- net A12: now also U7.2 (A12)
- net A13: now also U7.26 (A13)
- net A14: now also U7.1 (A14), U7.22 (~{OE})
- net A2: now also U7.8 (A2)
- net A3: now also U7.7 (A3)
- net A4: now also U7.6 (A4)
- net A5: now also U7.5 (A5)
- net A6: now also U7.4 (A6)
- net A7: now also U7.3 (A7)
- net A8: now also U7.25 (A8)
- net A9: now also U7.24 (A9)
- net D0: now also U7.11 (Q0)
- net D1: now also U7.12 (Q1)
- net D2: now also U7.13 (Q2)
- net D3: now also U7.15 (Q3)
- net D4: now also U7.16 (Q4)
- net D5: now also U7.17 (Q5)
- net D6: now also U7.18 (Q6)
- net D7: now also U7.19 (Q7)
- net GND: now also U1.E2 (AVEC), U2.7 (GND), U7.14 (GND)
- net RESET: now also U2.1 (~{R})
- net R~{W}: now also U7.27 (~{WE})
- net at SW1.2, U1.F12 (RESET): no longer U1.H2 (HLT)
- net FC1: now reaches U1.C1 (FC1)
- net FC2: now reaches U1.D1 (FC2)
- net FC0: now reaches U1.D2 (FC0)
- net DSACK0: now reaches U1.F1 (DSACK0)
- net STERM: now reaches U1.G1 (STERM)
- net IPL2: now reaches U1.G12 (IPL2)
- net IPL1: now reaches U1.G13 (IPL1)
- net DSACK1: now reaches U1.G2 (DSACK1)
- net AS: now reaches U1.J2 (AS)
- net DS: now reaches U1.K2 (DS)
- net SIZ1: now reaches U1.K3 (SIZ1)
- net SIZ0: now reaches U1.L2 (SIZ0)
- net ECS: now reaches U1.M2 (ECS)
- net ECS: now also U2.3 (C)
- new net: JP1.1 (A), U1.H2 (HLT)
- new net: JP1.2 (B), U2.5 (Q)
- new net: R8.2, U2.4 (~{S})
- new net: U2.2 (D), U2.6 (~{Q})
- new net RAM0: U7.20 (~{CS})
- no-connect marks 15 -> 17
Other:
- added sheet GLUE Logic (glue.kicad_sch)
- added sheet Graphical Interface Bus (gib.kicad_sch)
- added sheet PCI (pci.kicad_sch)

Commit message: ygffd
Parts:
- added R10, R9: 10k, Resistor_SMD:R_0603_1608Metric, symbol Device:R_US
Connections:
- net +5V: now also R10.1, R9.1
- net GND: no longer U1.E2 (AVEC)
- net DSACK0: no longer names the net of U1.F1 (DSACK0)
- net DSACK0: now also R9.2
- net DSACK1: no longer names the net of U1.G2 (DSACK1)
- net DSACK1: now also R10.2
- net ECS: no longer names the net of U1.M2 (ECS)
- net ECS: no longer U2.3 (C)
- net IPL1: no longer names the net of U1.G13 (IPL1)
- net IPL2: no longer names the net of U1.G12 (IPL2)
- new net VERA/IRQ: U1.E2 (AVEC)
- no-connect marks 17 -> 40
Other:
- removed sheet Graphical Interface Bus
- added sheet VERA (vera.kicad_sch)
