File: kicad/main/cpu.kicad_sch (KiCad schematic)
At the start: 14 parts, among them SW1 SW_Push, U1 MC68030RC_PGA, U13 28C256, U2 74HC74, U7 CY62256-70PC, Y1 CXO_DIP8

Commit message: more stuff
added support for the VERA module in the emulator
also re-doing the PCB

Co-Authored-By: Claude <claude@users.noreply.github.com>
Parts:
- removed JP1: RUN, TestPoint:TestPoint_2Pads_Pitch5.08mm_Drill1.3mm, symbol Jumper:Jumper_2_Open
- removed R1, R2, R3, R4, R5, R6, R8: 10k, Resistor_SMD:R_1206_3216Metric, symbol Device:R_US
- removed SW1: SW_Push, Button_Switch_THT:SW_PUSH_6mm, symbol Switch:SW_Push
- removed U1: MC68030RC_PGA, cpu:MC68030, symbol cpu:MC68030RC_PGA
- removed U13: 28C256, Package_DIP:DIP-28_W15.24mm_LongPads, symbol Memory_EEPROM:28C256
- removed U2: 74HC74, Package_DIP:DIP-14_W7.62mm_LongPads, symbol 74xx:74HC74
- removed U7: CY62256-70PC, Package_DIP:DIP-28_W15.24mm, symbol Memory_RAM:CY62256-70PC
- removed Y1: CXO_DIP8, Oscillator:Oscillator_DIP-8_LargePads, symbol Oscillator:CXO_DIP8
- added U1: MC68030RC_PGA, az030:MC68030, symbol az030:MC68030RC_PGA
- added U2: CY62256-70PC, Package_DIP:DIP-28_W15.24mm_LongPads, symbol Memory_RAM:CY62256-70PC
Connections:
- net +5V: now also U1.C6 (VCC), U1.D10 (VCC), U1.D4 (VCC), U1.F11 (VCC), U1.F2 (VCC), U1.H11 (VCC), U1.H3 (VCC), U1.K10 (VCC), U1.K4 (VCC), U1.L6 (VCC)
- net GND: now also U1.C5 (GND), U1.C7 (GND), U1.C9 (GND), U1.E11 (GND), U1.E3 (GND), U1.F3 (GND), U1.G11 (GND), U1.G3 (GND), U1.J11 (GND), U1.J3 (GND), U1.L5 (GND), U1.L7 (GND), U1.L8 (GND), U1.L9 (GND)
- no-connect marks 17 -> 0
Other:
- removed sheet GLUE Logic
- removed sheet Graphical Interface Bus
- removed sheet PCI
- title: CPU -> (none)
