File: kicad/main/cpu.kicad_sch (KiCad schematic)
At the start: 2 parts, among them U1 MC68030RC_PGA, U2 CY62256-70PC

Commit message: yuh
Parts:
- added U4: 74AHC1G04, Package_TO_SOT_SMD:SOT-553, symbol 74xGxx:74AHC1G04
Connections:
- net +5V: now also U2.28 (VCC), U4.5 (VCC)
- net GND: now also U2.14 (GND), U4.3 (GND)
- net RAM0: now reaches U2.20 (~{CS})
- net ~{R}/W: now reaches U2.22 (~{OE})
- net ~{R}/W: now also U4.4
- net R/~{W}: now reaches U2.27 (~{WE})
- net R/~{W}: now also U1.L3 (R_W), U4.2
- net DSACK0: now reaches U1.F1 (DSACK0)
- net DSACK1: now reaches U1.G2 (DSACK1)
Other:
- added sheet glue (glue.kicad_sch)

Commit message: gonna see if i can switch back to linux
Parts:
- added C5: 0u1, symbol Device:C
- added R1: 1k, Resistor_THT:R_Axial_DIN0204_L3.6mm_D1.6mm_P5.08mm_Horizontal, symbol Device:R_US
- added SW1: SW_Push, Button_Switch_THT:SW_PUSH_6mm, symbol Switch:SW_Push
- added U5: 28C256, Package_DIP:DIP-28_W15.24mm_Socket_LongPads, symbol Memory_EEPROM:28C256
Connections:
- net +5V: now also U5.27 (~{WE}), U5.28 (VCC)
- net GND: now also C5.2, SW1.1, U5.14 (GND), U5.22 (~{OE})
- net RESET: now reaches U1.F12 (RESET)
- net RESET: now also C5.1, R1.2, SW1.2
- new net RESET_FP: R1.1
- new net ROM: U5.20 (~{CS})
