File: kicad/main/gib.kicad_sch (KiCad schematic)
At the start: 1 part

Commit message: ygffd
Parts:
- removed U9: (no value), Connector_PCBEdge:Samtec_MECF-40-01-L-DV-WT_2x40_P1.27mm_Polarized_Socket_Horizontal, symbol az030_Symbols:GIB_Connector_Fem
Connections:
- no-connect marks 2 -> 0
