File: kicad/main/glue.kicad_sch (KiCad schematic)
At the start: 0 parts

Commit message: so much shit done holy
Parts:
- added C1, C3: 100n, Capacitor_SMD:C_0201_0603Metric, symbol Device:C
- added C2: 10u, Capacitor_SMD:C_0201_0603Metric, symbol Device:C
- added J8: Conn_01x04_Pin, Connector_PinHeader_2.54mm:PinHeader_1x04_P2.54mm_Vertical, symbol Connector:Conn_01x04_Pin
- added U5: XC9572XL-10VQG64C, Package_QFP:TQFP-64_10x10mm_P0.5mm, symbol CPLD_Xilinx:XC9572XL-xxVQx64
Connections:
- new net: C2.1, U5.26 (VCCIO), U5.55 (VCCIO)
- new net: C1.1, U5.3 (VCCINT), U5.37 (VCCINT)
- new net: C3.1, U5.14 (GND), U5.21 (GND), U5.41 (GND), U5.54 (GND)
- new net: J8.1 (Pin_1), U5.30 (TCK)
- new net: J8.2 (Pin_2), U5.28 (TDI)
- new net: J8.3 (Pin_3), U5.53 (TDO)
- new net: J8.4 (Pin_4), U5.29 (TMS)
- new net +3.3V: C1.2, C2.2
- new net GND: C3.2
Other:
- title: (none) -> GLUE Logic

Commit message: fjfjkdsldkjjfds
Parts:
- removed C1, C3: 100n, Capacitor_SMD:C_0201_0603Metric, symbol Device:C
- removed C2: 10u, Capacitor_SMD:C_0201_0603Metric, symbol Device:C
- removed J8: Conn_01x04_Pin, Connector_PinHeader_2.54mm:PinHeader_1x04_P2.54mm_Vertical, symbol Connector:Conn_01x04_Pin
- removed U5: XC9572XL-10VQG64C, Package_QFP:TQFP-64_10x10mm_P0.5mm, symbol CPLD_Xilinx:XC9572XL-xxVQx64
- added U5, U6: GAL16V8, Package_DIP:DIP-20_W7.62mm_LongPads, symbol Logic_Programmable:GAL16V8
Connections:
- net GND: now also U5.10 (GND), U6.10 (GND)
- new net +5V: U5.20 (V_{CC}), U6.20 (V_{CC})
- new net A0: U5.2 (I_{1})
- new net A1: U5.1 (I_{0})
- new net A19: U5.3 (I_{2})
- new net A20: U5.4 (I_{3})
- new net A25: U5.5 (I_{4}), U6.3 (I_{2})
- new net AS: U5.8 (I_{7})
- new net CLOCK: U6.1 (I_{0})
- new net DSACK0: U6.12 (F_{0})
- new net DSACK1: U6.13 (F_{1})
- new net EXT: U5.19 (F_{7})
- new net RAM0: U5.13 (F_{1})
- new net RAM1: U5.14 (F_{2})
- new net RAM2: U5.15 (F_{3})
- new net RAM3: U5.16 (F_{4})
- new net ROM: U5.17 (F_{5})
- new net R/~{W}: U6.2 (I_{1})
- new net SIZ0: U5.6 (I_{5})
- new net SIZ1: U5.7 (I_{6})
- new net STERM: U6.14 (F_{2})
- new net UART: U5.18 (F_{6})
- no-connect marks 0 -> 4

Commit message: ygffd
Parts:
- removed U5, U6: GAL16V8, Package_DIP:DIP-20_W7.62mm_LongPads, symbol Logic_Programmable:GAL16V8
Connections:
- no-connect marks 4 -> 0
