File: kicad/main/glue.kicad_sch (KiCad schematic)
At the start: 5 parts, among them U3 ATF1502AS-xAx44

Commit message: gonna see if i can switch back to linux
Connections:
- net +5V: now also U3.17 (VCC), U3.29 (VCC), U3.41 (VCC), U3.9 (VCC)
- net GND: no longer U3.17 (VCC), U3.29 (VCC), U3.41 (VCC), U3.9 (VCC)
Changed lines of the file:
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@@
 	)
 	(junction
-		(at 74.93 64.77)
+		(at 40.64 57.15)
 		(diameter 0)
 		(color 0 0 0 0)
 	)
 	(junction
-		(at 40.64 57.15)
+		(at 74.93 57.15)
 		(diameter 0)
 		(color 0 0 0 0)
@@
 	(wire
 		(pts
-			(xy 113.03 64.77) (xy 113.03 77.47)
+			(xy 113.03 57.15) (xy 113.03 77.47)
 		)
 		(stroke
@@
 	(wire
 		(pts
-			(xy 74.93 64.77) (xy 113.03 64.77)
+			(xy 113.03 57.15) (xy 74.93 57.15)
 		)
 		(stroke
