File: kicad/main/io.kicad_sch (KiCad schematic)
At the start: 2 parts, among them J8 DE9_Pins_MountingHoles, J9 DB25_Pins_MountingHoles

Commit message: remove some stuff
Parts:
- removed J9: DB25_Pins_MountingHoles, Connector_Dsub:DSUB-25_Pins_Horizontal_P2.77x2.84mm_EdgePinOffset4.94mm_Housed_MountingHolesOffset4.94mm, symbol Connector:DB25_Pins_MountingHoles
- added J11: PS/2, Footprints:Connector_Mini-DIN_Female_6Pin_2rows, symbol Connector:Mini-DIN-6
- added U10: 74AHC595, Package_DIP:DIP-16_W7.62mm_LongPads, symbol 74xx:74AHC595
- added U11: 74AHC04, Package_DIP:DIP-14_W7.62mm_LongPads, symbol 74xx:74AHC04
Connections:
- new net: U10.11 (SRCLK), U11.2, U11.3
- new net: U11.4, U11.5
- new net: U10.12 (RCLK), U11.6
- new net +5V: J11.4, U10.10 (~{SRCLR}), U10.16 (VCC), U11.14 (VCC)
- new net GND: J11.3, U10.13 (~{OE}), U10.8 (GND), U11.7 (GND)
- new net PS/2 Clock: J11.5, U11.1
- new net PS/2 D0: U10.15 (QA)
- new net PS/2 D1: U10.1 (QB)
- new net PS/2 D2: U10.2 (QC)
- new net PS/2 D3: U10.3 (QD)
- new net PS/2 D4: U10.4 (QE)
- new net PS/2 D5: U10.5 (QF)
- new net PS/2 D6: U10.6 (QG)
- new net PS/2 D7: U10.7 (QH)
- new net PS/2 Data: J11.1, U10.14 (SER)
- no-connect marks 0 -> 3
Other:
- added sheet RS232 (rs232.kicad_sch)
