File: kicad/main/io.kicad_sch (KiCad schematic)
At the start: 4 parts, among them J11 PS/2, J8 DE9_Pins_MountingHoles, U10 74AHC595, U11 74AHC04

Commit message: more stuff
added support for the VERA module in the emulator
also re-doing the PCB

Co-Authored-By: Claude <claude@users.noreply.github.com>
Parts:
- removed J11: PS/2, Footprints:Connector_Mini-DIN_Female_6Pin_2rows, symbol Connector:Mini-DIN-6
- removed J8: DE9_Pins_MountingHoles, Connector_Dsub:DSUB-9_Pins_Horizontal_P2.77x2.84mm_EdgePinOffset4.94mm_Housed_MountingHolesOffset4.94mm, symbol Connector:DE9_Pins_MountingHoles
- removed U10: 74AHC595, Package_DIP:DIP-16_W7.62mm_LongPads, symbol 74xx:74AHC595
- removed U11: 74AHC04, Package_DIP:DIP-14_W7.62mm_LongPads, symbol 74xx:74AHC04
- added J3: DE9_Pins_MountingHoles, Connector_Dsub:DSUB-9_Pins_Horizontal_P2.77x2.84mm_EdgePinOffset4.94mm_Housed_MountingHolesOffset4.94mm, symbol Connector:DE9_Pins_MountingHoles
- added J4: DE15_Socket_HighDensity_MountingHoles, Connector_Dsub:DSUB-15_Socket_Horizontal_P2.77x2.84mm_EdgePinOffset4.94mm_Housed_MountingHolesOffset4.94mm, symbol Connector:DE15_Socket_HighDensity_MountingHoles
Connections:
- net GND: now also J3.SH (PAD), J4.SH
- no-connect marks 3 -> 24
Other:
- removed sheet RS232
- title: (none) -> Input and Output
