File: kicad/main/misc.kicad_sch (KiCad schematic)
At the start: 4 parts, among them J4 Conn_01x03_Pin, J5 Conn_01x03_Pin, J6 Conn_01x03_Pin, J7 Conn_01x03_Pin

Commit message: ygffd
Parts:
- removed J4, J5, J6, J7: Conn_01x03_Pin, Connector:FanPinHeader_1x03_P2.54mm_Vertical, symbol Connector:Conn_01x03_Pin
Connections:
- no-connect marks 4 -> 0
