File: kicad/main/pci.kicad_sch (KiCad schematic)
At the start: 1 part, among them J10 Bus_PCI_32bit_Universal

Commit message: ygffd
Parts:
- removed J10: Bus_PCI_32bit_Universal, Connector_PCBEdge:Samtec_MECF-60-01-L-DV-WT_2x60_P1.27mm_Polarized_Socket_Horizontal, symbol Connector:Bus_PCI_32bit_Universal
