File: kicad/main/perMan.kicad_sch (KiCad schematic)
At the start: 2 parts, among them U3 W65C22SxP, U4 W65C22SxP

Commit message: guhdwhudsa
Connections:
- net R~{W}: now reaches U3.22 (R/~{W})
- net R~{W}: now also U4.22 (R/~{W})
Changed lines of the file:
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@@
+	(wire
+		(pts
+			(xy 87.63 137.16) (xy 92.71 137.16)
+		)
+		(stroke
+			(width 0)
+			(type default)
+		)
+	)
 	(wire
 		(pts
@@
 		)
 	)
+	(wire
+		(pts
+			(xy 143.51 135.89) (xy 151.13 135.89)
+		)
+		(stroke
+			(width 0)
+			(type default)
+		)
+	)
+	(label "R~{W}"
+		(at 143.51 135.89 180)
+		(effects
+			(font
+				(size 1.27 1.27)
+			)
+			(justify right bottom)
+		)
+	)
+	(label "R~{W}"
+		(at 87.63 137.16 180)
+		(effects
+			(font
+				(size 1.27 1.27)
+			)
+			(justify right bottom)
+		)
+	)

Commit message: so much shit done holy
Other:
- title: (none) -> Peripheral Management
Changed lines of the file:
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@@
 	(paper "A3")
 	(title_block
-		(date "2026-10-06")
+		(title "Peripheral Management")
+		(date "2026-10-07")
 		(rev "A0001")
 		(company "azalea68k")

Commit message: ygffd
Parts:
- removed U3, U4: W65C22SxP, Package_DIP:DIP-40_W15.24mm, symbol 65xx-library:W65C22SxP
