File: kicad/main/power.kicad_sch (KiCad schematic)
At the start: 1 part

Commit message: so much shit done holy
Parts:
- removed D2: D_Schottky, Package_DFN_QFN:WDFN-10-1EP_3x3mm_P0.5mm_EP1.8x2.5mm, symbol Device:D_Schottky
- added F2: 5a, Fuse:Fuse_Blade_ATO_directSolder, symbol Device:Fuse
- added F3, F4: 3a, Fuse:Fuse_Blade_ATO_directSolder, symbol Device:Fuse
- added J1: ATX-24, Connector_Molex:Molex_Mini-Fit_Jr_5569-24A2_2x12_P4.20mm_Horizontal, symbol Connector:ATX-24
- added J2: Conn_01x02_Pin, Connector_PinHeader_2.54mm:PinHeader_1x02_P2.54mm_Vertical, symbol Connector:Conn_01x02_Pin
- added J3: LED, Connector_PinHeader_2.54mm:PinHeader_1x02_P2.54mm_Vertical, symbol Connector:Conn_01x02_Pin
- added R7: 330, Resistor_THT:R_Axial_DIN0204_L3.6mm_D1.6mm_P7.62mm_Horizontal, symbol Device:R_US
Connections:
- new net: F3.1, J1.1 (+3.3V), J1.12 (+3.3V), J1.13 (+3.3V), J1.2 (+3.3V)
- new net: F4.1, J1.10 (+12V), J1.11 (+12V)
- new net: F2.1, J1.21 (+5V), J1.22 (+5V), J1.23 (+5V), J1.4 (+5V), J1.6 (+5V)
- new net: J3.1 (Pin_1), R7.1
- new net: J1.8 (PWR_OK), J3.2 (Pin_2)
- new net: J1.16 (PS_ON#), J2.1 (Pin_1)
- new net +12V: F4.2
- new net +3.3V: F3.2
- new net +5V: F2.2
- new net GND: J1.15 (GND), J1.17 (GND), J1.18 (GND), J1.19 (GND), J1.24 (GND), J1.3 (GND), J1.5 (GND), J1.7 (GND), J2.2 (Pin_2), R7.2
- no-connect marks 0 -> 2
Other:
- title: (none) -> Power

Commit message: ygffd
Parts:
- removed F3, F4: 3a, Fuse:Fuse_Blade_ATO_directSolder, symbol Device:Fuse
Connections:
- no-connect marks 2 -> 4
