File: kicad/main/scsi.kicad_sch (KiCad schematic)
At the start: 3 parts

Commit message: fjfjkdsldkjjfds
Parts:
- removed D1: 1n4001, Diode_THT:D_DO-41_SOD81_P10.16mm_Horizontal, symbol Device:D
- removed F1: 1a, Fuse:Fuse_Littelfuse-LVR100, symbol Device:Fuse
- removed U2: (no value), Connector_IDC:IDC-Header_2x25_P2.54mm_Horizontal, symbol az030_Symbols:SCSI_50p_Internal
- added U8: (no value), Package_DIP:DIP-48_W15.24mm_LongPads, symbol az030_Symbols:Z53C80
Connections:
- new net RESET: U8.2 (RST)

Commit message: ygffd
Parts:
- removed U8: (no value), Package_DIP:DIP-48_W15.24mm_LongPads, symbol az030_Symbols:Z53C80
Changed lines of the file:
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@@
 		(comment 2 "based on the macintosh se/30's scsi implementation")
 	)
-	(wire
-		(pts
-			(xy 151.13 104.14) (xy 147.32 104.14)
-		)
-		(stroke
-			(width 0)
-			(type default)
-		)
-	)
-	(global_label "RESET"
-		(shape input)
-		(at 151.13 104.14 0)
-		(fields_autoplaced yes)
-		(effects
-			(font
-				(size 1.27 1.27)
-			)
-			(justify left)
-		)
-		(property "Intersheetrefs" "${INTERSHEET_REFS}"
-			(at 159.8603 104.14 0)
-			(hide yes)
-			(show_name no)
-			(do_not_autoplace no)
-			(effects
-				(font
-					(size 1.27 1.27)
-				)
-				(justify left)
-			)
-		)
-	)
-	(symbol
-		(lib_id "az030_Symbols:Z53C80")
-		(at 137.16 55.88 0)
-		(unit 1)
-		(body_style 1)
-		(exclude_from_sim no)
-		(in_bom yes)
-		(on_board yes)
-		(in_pos_files yes)
-		(dnp no)
-		(fields_autoplaced yes)
-		(property "Reference" "U8"
-			(at 136.525 132.08 0)
-			(show_name no)
-			(do_not_autoplace no)
-			(effects
-				(font
-					(size 1.27 1.27)
-				)
-			)
-		)
-		(property "Value" ""
-			(at 137.16 55.88 0)
-			(show_name no)
-			(do_not_autoplace no)
-			(effects
-				(font
-					(size 1.27 1.27)
-				)
-			)
-		)
-		(property "Footprint" "Package_DIP:DIP-48_W15.24mm_LongPads"
-			(at 137.16 55.88 0)
-			(hide yes)
-			(show_name no)
-			(do_not_autoplace no)
-			(effects
-				(font
-					(size 1.27 1.27)
-				)
-			)
-		)
-		(property "Datasheet" ""
-			(at 137.16 55.88 0)
-			(hide yes)
-			(show_name no)
-			(do_not_autoplace no)
-			(effects
-				(font
-					(size 1.27 1.27)
-				)
-			)
-		)
-		(property "Description" ""
-			(at 137.16 55.88 0)
-			(hide yes)
-			(show_name no)
-			(do_not_autoplace no)
-			(effects
-				(font
-					(size 1.27 1.27)
-				)
-			)
-		)
-		(pin "12"
-		)
-		(pin "20"
-		)
-		(pin "19"
-		)
-		(pin "17"
-		)
-		(pin "9"
-		)
-		(pin "8"
-		)
-		(pin "44"
-		)
-		(pin "37"
-		)
-		(pin "20"
-		)
-		(pin "38"
-		)
-		(pin "48"
-		)
-		(pin "45"
-		)
-		(pin "14"
-		)
-		(pin "33"
-		)
-		(pin "41"
-		)
-		(pin "2"
-		)
-		(pin "40"
-		)
-		(pin "1"
-		)
-		(pin "30"
-		)
-		(pin "32"
-		)
-		(pin "29"
-		)
-		(pin "43"
-		)
-		(pin "21"
-		)
-		(pin "16"
-		)
-		(pin "15"
-		)
-		(pin "47"
-		)
-		(pin "6"
-		)
-		(pin "4"
-		)
-		(pin "27"
-		)
-		(pin "26"
-		)
-		(pin "25"
-		)
-		(pin "36"
-		)
-		(pin "35"
-		)
-		(pin "11"
-		)
-		(pin "22"
-		)
-		(pin "28"
-		)
-		(pin "10"
-		)
-		(pin "5"
-		)
-		(pin "21"
-		)
-		(instances
-			(project "az030"
-				(path "/23b23725-f42e-4e44-9db5-2c9059cb0f3d/d4625fa3-dde9-4bfa-92c4-31e1384a32e2"
-					(reference "U8")
-					(unit 1)
-				)
-			)
-		)
-	)
 )
