File: kicad/main/scsi.kicad_sch (KiCad schematic)
At the start: 1 part

Commit message: more stuff
added support for the VERA module in the emulator
also re-doing the PCB

Co-Authored-By: Claude <claude@users.noreply.github.com>
Parts:
- removed U8: (no value), Package_DIP:DIP-48_W15.24mm_LongPads, symbol az030_Symbols:Z53C80
- added UI1: 53C80, Package_LCC:PLCC-44_16.6x16.6mm_P1.27mm, symbol az030:53C80
Other:
- title: SCSI Implementation -> (none)
Changed lines of the file:
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@@
 	(paper "A4")
 	(title_block
-		(title "SCSI Implementation")
-		(date "2026-10-07")
+		(date "2026-10-14")
 		(rev "A0001")
 		(company "azalea68k")
-		(comment 1 "revision format: Axxxx")
-		(comment 2 "based on the macintosh se/30's scsi implementation")
 	)
-	(wire
-		(pts
-			(xy 151.13 104.14) (xy 147.32 104.14)
-		)
-		(stroke
-			(width 0)
-			(type default)
-		)
-	)
-	(global_label "RESET"
-		(shape input)
-		(at 151.13 104.14 0)
+	(symbol
+		(lib_id "az030:53C80")
+		(at 97.79 69.85 0)
+		(unit 1)
+		(body_style 1)
+		(exclude_from_sim no)
+		(in_bom yes)
+		(on_board yes)
+		(in_pos_files yes)
+		(dnp no)
 		(fields_autoplaced yes)
-		(effects
-			(font
-				(size 1.27 1.27)
-			)
-			(justify left)
-		)
-		(property "Intersheetrefs" "${INTERSHEET_REFS}"
-			(at 159.8603 104.14 0)
-			(hide yes)
+		(property "Reference" "UI1"
+			(at 99.9333 39.37 0)
 			(show_name no)
 			(do_not_autoplace no)
@@
 			)
 		)
-	)
-	(symbol
-		(lib_id "az030_Symbols:Z53C80")
-		(at 137.16 55.88 0)
-		(unit 1)
-		(body_style 1)
-		(exclude_from_sim no)
-		(in_bom yes)
-		(on_board yes)
-		(in_pos_files yes)
-		(dnp no)
-		(fields_autoplaced yes)
-		(property "Reference" "U8"
-			(at 136.525 132.08 0)
+		(property "Value" "53C80"
+			(at 99.9333 41.91 0)
 			(show_name no)
 			(do_not_autoplace no)
@@
 					(size 1.27 1.27)
 				)
+				(justify left)
 			)
 		)
-		(property "Value" ""
-			(at 137.16 55.88 0)
-			(show_name no)
-			(do_not_autoplace no)
-			(effects
-				(font
-					(size 1.27 1.27)
-				)
-			)
-		)
-		(property "Footprint" "Package_DIP:DIP-48_W15.24mm_LongPads"
-			(at 137.16 55.88 0)
+		(property "Footprint" "Package_LCC:PLCC-44_16.6x16.6mm_P1.27mm"
+			(at 97.79 69.85 0)
 			(hide yes)
 			(show_name no)
@@
 		)
 		(property "Datasheet" ""
-			(at 137.16 55.88 0)
+			(at 97.79 69.85 0)
 			(hide yes)
 			(show_name no)
@@
 		)
 		(property "Description" ""
-			(at 137.16 55.88 0)
+			(at 97.79 69.85 0)
 			(hide yes)
 			(show_name no)
@@
 			)
 		)
-		(pin "12"
+		(pin "44"
 		)
-		(pin "20"
+		(pin "43"
+		)
+		(pin "41"
+		)
+		(pin "42"
+		)
+		(pin "40"
+		)
+		(pin "39"
+		)
+		(pin "29"
+		)
+		(pin "8"
+		)
+		(pin "7"
+		)
+		(pin "9"
+		)
+		(pin "6"
 		)
 		(pin "19"
 		)
-		(pin "17"
+		(pin "10"
 		)
-		(pin "9"
+		(pin "12"
 		)
-		(pin "8"
+		(pin "11"
 		)
-		(pin "44"
+		(pin "15"
+		)
+		(pin "14"
+		)
+		(pin "1"
+		)
+		(pin "2"
+		)
+		(pin "4"
+		)
+		(pin "5"
+		)
+		(pin "3"
+		)
+		(pin "31"
+		)
+		(pin "34"
+		)
+		(pin "35"
+		)
+		(pin "36"
+		)
+		(pin "33"
+		)
+		(pin "32"
 		)
 		(pin "37"
+		)
+		(pin "28"
+		)
+		(pin "26"
+		)
+		(pin "27"
+		)
+		(pin "25"
+		)
+		(pin "24"
+		)
+		(pin "23"
+		)
+		(pin "22"
+		)
+		(pin "21"
+		)
+		(pin "30"
+		)
+		(pin "13"
 		)
 		(pin "20"
@@
 		(pin "38"
 		)
-		(pin "48"
-		)
-		(pin "45"
-		)
-		(pin "14"
-		)
-		(pin "33"
-		)
-		(pin "41"
-		)
-		(pin "2"
-		)
-		(pin "40"
-		)
-		(pin "1"
-		)
-		(pin "30"
-		)
-		(pin "32"
-		)
-		(pin "29"
-		)
-		(pin "43"
-		)
-		(pin "21"
-		)
 		(pin "16"
 		)
-		(pin "15"
+		(pin "18"
 		)
-		(pin "47"
-		)
-		(pin "6"
-		)
-		(pin "4"
-		)
-		(pin "27"
-		)
-		(pin "26"
-		)
-		(pin "25"
-		)
-		(pin "36"
-		)
-		(pin "35"
-		)
-		(pin "11"
-		)
-		(pin "22"
-		)
-		(pin "28"
-		)
-		(pin "10"
-		)
-		(pin "5"
-		)
-		(pin "21"
+		(pin "17"
 		)
 		(instances
-			(project "az030"
-				(path "/23b23725-f42e-4e44-9db5-2c9059cb0f3d/d4625fa3-dde9-4bfa-92c4-31e1384a32e2"
-					(reference "U8")
+			(project "main"
+				(path "/49283a4e-28ec-4bf4-b38a-36a5ba9c2baf/d57c9ca3-ae9b-4906-a9d1-d8fc30f0c86c/9290ec60-0e52-4186-b6db-73cde75f92ba"
+					(reference "UI1")
 					(unit 1)
 				)
