File: kicad/main/main.kicad_pcb (KiCad board)
At the start: 2 copper layers, 304.8 x 243.8 mm, 7 parts, among them J1 ATX-24, J2 Conn_01x02_Pin, J3 DE9_Pins_MountingHoles, J4 DE15_Socket_HighDensity_Mount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, U1 MC68030RC_PGA

Commit message: yuh
Parts:
- added C1: 100n, Capacitor_SMD:C_0603_1608Metric, F.Cu at (353.3, 208.5)
- added C2: 100n, Capacitor_SMD:C_0603_1608Metric, F.Cu at (350.8, 208.5)
- added C3: 100n, Capacitor_SMD:C_0603_1608Metric, F.Cu at (348.3, 208.5)
- added C4: 100n, Capacitor_SMD:C_0603_1608Metric, F.Cu at (345.8, 208.5)
- added U2: CY62256-70PC, Package_DIP:DIP-28_W15.24mm_LongPads, F.Cu at (388.3, 219.8)
- added U3: ATF1502AS-xAx44, Package_QFP:TQFP-44_10x10mm_P0.8mm, F.Cu at (347.4, 199.3)
- added U4: 74AHC1G04, Package_TO_SOT_SMD:SOT-553, F.Cu at (372.0, 238.0)
- turned U1 to -90 degrees
Connections:
- U1 pad A10: unconnected-(U1-A17-PadA10) -> /cpu/A17
- U1 pad A11: unconnected-(U1-A15-PadA11) -> /cpu/A15
- U1 pad A12: unconnected-(U1-A13-PadA12) -> /cpu/A13
- U1 pad A13: unconnected-(U1-A10-PadA13) -> /cpu/A10
- U1 pad A2: unconnected-(U1-A0-PadA2) -> /cpu/A0
- U1 pad A3: unconnected-(U1-A30-PadA3) -> /cpu/A30
- U1 pad A4: unconnected-(U1-A28-PadA4) -> /cpu/A28
- U1 pad A5: unconnected-(U1-A26-PadA5) -> /cpu/A26
- U1 pad A6: unconnected-(U1-A24-PadA6) -> /cpu/A24
- U1 pad A7: unconnected-(U1-A23-PadA7) -> /cpu/A23
- U1 pad A8: unconnected-(U1-A21-PadA8) -> /cpu/A21
- U1 pad A9: unconnected-(U1-A19-PadA9) -> /cpu/A19
- U1 pad B10: unconnected-(U1-A14-PadB10) -> /cpu/A14
- U1 pad B11: unconnected-(U1-A12-PadB11) -> /cpu/A12
- U1 pad B12: unconnected-(U1-A8-PadB12) -> /cpu/A8
- U1 pad B13: unconnected-(U1-A7-PadB13) -> /cpu/A7
- U1 pad B3: unconnected-(U1-A31-PadB3) -> /cpu/A31
- U1 pad B4: unconnected-(U1-A29-PadB4) -> /cpu/A29
- U1 pad B5: unconnected-(U1-A27-PadB5) -> /cpu/A27
- U1 pad B6: unconnected-(U1-A25-PadB6) -> /cpu/A25
- U1 pad B7: unconnected-(U1-A22-PadB7) -> /cpu/A22
- U1 pad B8: unconnected-(U1-A20-PadB8) -> /cpu/A20
- U1 pad B9: unconnected-(U1-A16-PadB9) -> /cpu/A16
- U1 pad C10: unconnected-(U1-A11-PadC10) -> /cpu/A11
- U1 pad C11: unconnected-(U1-A9-PadC11) -> /cpu/A9
- U1 pad C12: unconnected-(U1-A5-PadC12) -> /cpu/A5
- U1 pad C13: unconnected-(U1-A4-PadC13) -> /cpu/A4
- U1 pad C4: unconnected-(U1-A1-PadC4) -> /cpu/A1
- U1 pad C5: unconnected-(U1-GND-PadC5) -> GND
- U1 pad C6: unconnected-(U1-VCC-PadC6) -> +5V
- U1 pad C7: unconnected-(U1-GND-PadC7) -> GND
- U1 pad C8: unconnected-(U1-A18-PadC8) -> /cpu/A18
- U1 pad C9: unconnected-(U1-GND-PadC9) -> GND
- U1 pad D10: unconnected-(U1-VCC-PadD10) -> +5V
- U1 pad D11: unconnected-(U1-A6-PadD11) -> /cpu/A6
- U1 pad D12: unconnected-(U1-A3-PadD12) -> /cpu/A3
- U1 pad D13: unconnected-(U1-A2-PadD13) -> /cpu/A2
- U1 pad D4: unconnected-(U1-VCC-PadD4) -> +5V
- U1 pad E11: unconnected-(U1-GND-PadE11) -> GND
- U1 pad E3: unconnected-(U1-GND-PadE3) -> GND
- U1 pad F1: unconnected-(U1-DSACK0-PadF1) -> DSACK0
- U1 pad F11: unconnected-(U1-VCC-PadF11) -> +5V
- U1 pad F2: unconnected-(U1-VCC-PadF2) -> +5V
- U1 pad F3: unconnected-(U1-GND-PadF3) -> GND
- U1 pad G11: unconnected-(U1-GND-PadG11) -> GND
- U1 pad G2: unconnected-(U1-DSACK1-PadG2) -> DSACK1
- U1 pad G3: unconnected-(U1-GND-PadG3) -> GND
- U1 pad H11: unconnected-(U1-VCC-PadH11) -> +5V
- U1 pad H3: unconnected-(U1-VCC-PadH3) -> +5V
- U1 pad J11: unconnected-(U1-GND-PadJ11) -> GND
- U1 pad J3: unconnected-(U1-GND-PadJ3) -> GND
- U1 pad K10: unconnected-(U1-VCC-PadK10) -> +5V
- U1 pad K11: unconnected-(U1-D5-PadK11) -> /cpu/D5
- U1 pad K12: unconnected-(U1-D1-PadK12) -> /cpu/D1
- U1 pad K13: unconnected-(U1-D0-PadK13) -> /cpu/D0
- U1 pad K4: unconnected-(U1-VCC-PadK4) -> +5V
- U1 pad L10: unconnected-(U1-D10-PadL10) -> /cpu/D10
- U1 pad L11: unconnected-(U1-D7-PadL11) -> /cpu/D7
- U1 pad L12: unconnected-(U1-D4-PadL12) -> /cpu/D4
- U1 pad L13: unconnected-(U1-D2-PadL13) -> /cpu/D2
- U1 pad L3: unconnected-(U1-R_W-PadL3) -> R/~{W}
- U1 pad L4: unconnected-(U1-D30-PadL4) -> /cpu/D30
- U1 pad L5: unconnected-(U1-GND-PadL5) -> GND
- U1 pad L6: unconnected-(U1-VCC-PadL6) -> +5V
- U1 pad L7: unconnected-(U1-GND-PadL7) -> GND
- U1 pad L8: unconnected-(U1-GND-PadL8) -> GND
- U1 pad L9: unconnected-(U1-GND-PadL9) -> GND
- U1 pad M10: unconnected-(U1-D12-PadM10) -> /cpu/D12
- U1 pad M11: unconnected-(U1-D9-PadM11) -> /cpu/D9
- U1 pad M12: unconnected-(U1-D6-PadM12) -> /cpu/D6
- U1 pad M13: unconnected-(U1-D3-PadM13) -> /cpu/D3
- U1 pad M3: unconnected-(U1-D29-PadM3) -> /cpu/D29
- U1 pad M4: unconnected-(U1-D27-PadM4) -> /cpu/D27
- U1 pad M5: unconnected-(U1-D24-PadM5) -> /cpu/D24
- U1 pad M6: unconnected-(U1-D22-PadM6) -> /cpu/D22
- U1 pad M7: unconnected-(U1-D20-PadM7) -> /cpu/D20
- U1 pad M8: unconnected-(U1-D17-PadM8) -> /cpu/D17
- U1 pad M9: unconnected-(U1-D14-PadM9) -> /cpu/D14
- U1 pad N1: unconnected-(U1-D31-PadN1) -> /cpu/D31
- U1 pad N10: unconnected-(U1-D15-PadN10) -> /cpu/D15
- U1 pad N11: unconnected-(U1-D13-PadN11) -> /cpu/D13
- U1 pad N12: unconnected-(U1-D11-PadN12) -> /cpu/D11
- U1 pad N13: unconnected-(U1-D8-PadN13) -> /cpu/D8
- U1 pad N2: unconnected-(U1-D28-PadN2) -> /cpu/D28
- U1 pad N3: unconnected-(U1-D26-PadN3) -> /cpu/D26
- U1 pad N4: unconnected-(U1-D25-PadN4) -> /cpu/D25
- U1 pad N5: unconnected-(U1-D23-PadN5) -> /cpu/D23
- U1 pad N6: unconnected-(U1-D21-PadN6) -> /cpu/D21
- U1 pad N7: unconnected-(U1-D19-PadN7) -> /cpu/D19
- U1 pad N8: unconnected-(U1-D18-PadN8) -> /cpu/D18
- U1 pad N9: unconnected-(U1-D16-PadN9) -> /cpu/D16
Routing:
- net R/~{W}: track 0.00 -> 17.0 mm
- net ~{R}/W: track 0.00 -> 3.88 mm
- net +5V: track 0.00 -> 2.92 mm, vias 0 -> 1
- net GND: track 23.2 -> 24.1 mm, vias 0 -> 1
- added copper zone on B.Cu, net +5V
- added copper zone on F.Cu, net GND

Commit message: gonna see if i can switch back to linux
Parts:
- removed J2: Conn_01x02_Pin, Connector_JST:JST_EH_B2B-EH-A_1x02_P2.50mm_Vertical
- added J5: ~, Connector_PinHeader_2.54mm:PinHeader_2x03_P2.54mm_Vertical, F.Cu at (145.0, 299.9)
- added R1: 1k, Resistor_THT:R_Axial_DIN0204_L3.6mm_D1.6mm_P5.08mm_Horizontal, F.Cu at (395.0, 199.5)
- added SW1: SW_Push, Button_Switch_THT:SW_PUSH_6mm, F.Cu at (399.5, 185.0)
- added U5: 28C256, Package_DIP:DIP-28_W15.24mm_Socket_LongPads, F.Cu at (354.5, 180.2)
- C1, C2, C3, C4: moved to B.Cu
- moved U2 37.2 mm to (354.5, 235.2), turned to 90 degrees
- moved U4 21.0 mm to (370.8, 217.0), turned to 180 degrees
- moved C1 10.5 mm to (351.6, 198.2), turned to 90 degrees
- moved C2 10.3 mm to (350.0, 198.2), turned to 90 degrees
- moved C4 10.3 mm to (345.1, 198.2), turned to 90 degrees
- moved C3 10.3 mm to (347.6, 198.2), turned to 90 degrees
Connections:
- J1 pad 8: unconnected-(J1-PWR_OK-Pad8) -> Net-(J1-PWR_OK)
- U1 pad F12: unconnected-(U1-RESET-PadF12) -> RESET
- U3 pad 17: GND -> +5V
- U3 pad 29: GND -> +5V
- U3 pad 41: GND -> +5V
- U3 pad 9: GND -> +5V
Routing:
- net RESET_FP: track 0.00 -> 340.1 mm
- net Net-(J1-PWR_OK): track 0.00 -> 284.9 mm
- net Net-(J1-PS_ON#): track 30.2 -> 313.0 mm
- net RESET: track 0.00 -> 28.7 mm
- net +5V: track 2.92 -> 28.2 mm, vias 1 -> 5
- net GND: track 24.1 -> 8.69 mm, vias 1 -> 5
